File: hardware/blanking_board/blanking_board.sch (KiCad schematic (older format))
At the start: 27 parts

Commit message: schematic update
Connections:
- net p1_chan4: now reaches J?.10
- net p1_chan5: now reaches J?.11
- net p1_chan6: now reaches J?.12
- net p1_chan1: now reaches J?.7
- net p1_chan2: now reaches J?.8
- net p1_chan3: now reaches J?.9
- net p2_chan4: now reaches J?.10
- net p2_chan5: now reaches J?.11
- net p2_chan6: now reaches J?.12
- net p2_chan1: now reaches J?.7
- net p2_chan2: now reaches J?.8
- net p2_chan3: now reaches J?.9
Changed lines of the file:
@@
 	0    1    1    0
 $EndComp
+Text GLabel 10350 2750 0    50   Input ~ 0
+p1_chan1
+Text GLabel 10350 2950 0    50   Input ~ 0
+p1_chan2
+Text GLabel 10350 3150 0    50   Input ~ 0
+p1_chan3
+Text GLabel 10350 3350 0    50   Input ~ 0
+p1_chan4
+Text GLabel 10350 3550 0    50   Input ~ 0
+p1_chan5
+Text GLabel 10350 3750 0    50   Input ~ 0
+p1_chan6
+Wire Wire Line
+	10350 2750 10600 2750
+Wire Wire Line
+	10350 2950 10600 2950
+Wire Wire Line
+	10350 3150 10600 3150
+Wire Wire Line
+	10350 3350 10600 3350
+Wire Wire Line
+	10350 3550 10600 3550
+Wire Wire Line
+	10350 3750 10600 3750
+Text GLabel 9650 5500 1    50   Input ~ 0
+p2_chan1
+Text GLabel 8650 5500 1    50   Input ~ 0
+p2_chan6
+Text GLabel 8850 5500 1    50   Input ~ 0
+p2_chan5
+Text GLabel 9050 5500 1    50   Input ~ 0
+p2_chan4
+Text GLabel 9250 5500 1    50   Input ~ 0
+p2_chan3
+Text GLabel 9450 5500 1    50   Input ~ 0
+p2_chan2
+Wire Wire Line
+	9650 5500 9650 5600
+Wire Wire Line
+	9450 5500 9450 5600
+Wire Wire Line
+	9250 5500 9250 5600
+Wire Wire Line
+	9050 5500 9050 5600
+Wire Wire Line
+	8850 5500 8850 5600
+Wire Wire Line
+	8650 5500 8650 5600
 $EndSCHEMATC

Commit message: update board
Parts:
- added J?: B4B-XH-A_LF__SN_, digikey-footprints:PinHeader_1x4_P2.5mm_Drill1.1mm, symbol dk_Rectangular-Connectors-Headers-Male-Pins:B4B-XH-A_LF__SN_
- added J? (x2): Conn_01x02_Female, symbol Connector:Conn_01x02_Female
- added JP?: Jumper_NC_Dual, symbol Device:Jumper_NC_Dual
Connections:
- net +5V: now also J?.3, J?.3, J?.3, J?.3, J?.3, J?.3, J?.3
- net at U?.1: now also J?.1 (x3)
- net blanking: now reaches U?.2
- net blanking: now also U?.10, U?.10, U?.10, U?.13, U?.13, U?.13, U?.2, U?.2, U?.5, U?.5, U?.5, JP?.2
- net at U?.4: now also J?.2 (x3)
- net at U?.9: now also J?.1 (x3)
- net at U?.12: now also J?.2 (x3)
- net GND: now reaches U?.7 (GND)
- net GND: now also J?.0 (PAD), J?.0 (PAD), J?.13, J?.13, J?.14 (P14), J?.14 (P14), J?.15 (P15), J?.15 (P15), J?.16 (P16), J?.16 (P16), J?.17 (P17), J?.17 (P17), J?.18 (P18), J?.18 (P18), J?.19 (P19), J?.19 (P19), J?.2, J?.20 (P20), J?.20 (P20), J?.21 (P21), J?.21 (P21), J?.22 (P22), J?.22 (P22), J?.23 (P23), J?.23 (P23), J?.24 (P24), J?.24 (P24), J?.25 (P25), J?.25 (P25), J?.4, J?.4, J?.4, J?.4, J?.4, J?.4, U?.7 (GND), U?.7 (GND), U?.7 (GND), J?.2 (Pin_2), J?.2 (Pin_2), J?.4
- net at R?.1, U?.1: now also JP?.3
- net at U?.2: now also JP?.1
- net at R?.2: now also J?.1
- new net: J?.1, J?.1 (Pin_1)
- new net: J?.1 (Pin_1), J?.2
- no-connect marks 0 -> 12
Other:
- moved on the sheet: J?, U?A, U?B, U?C, U?D, U?E

Commit message: first version of PCB
Parts:
- added H1, H2, H3, H4: MountingHole, MountingHole:MountingHole_3.2mm_M3_ISO7380, symbol Mechanical:MountingHole
- J1, J2, J3, J5, J6, J7, J8: renamed from J?; footprint digikey-footprints:PinHeader_1x4_P2.5mm_Drill1.1mm -> Connector_JST:JST_XH_B4B-XH-A_1x04_P2.50mm_Vertical
- J10, J9: renamed from J?; footprint (none) -> Connector_JST:JST_XH_B2B-XH-A_1x02_P2.50mm_Vertical
- J11, J12: renamed from J?; footprint (none) -> Connector_PinHeader_2.54mm:PinHeader_2x13_P2.54mm_Vertical
- J4: renamed from J?; footprint digikey-footprints:PinHeader_1x2_P2.5mm_Drill1.1mm -> Connector_JST:JST_XH_B2B-XH-A_1x02_P2.50mm_Vertical
- JP1: renamed from JP?; footprint (none) -> Connector_PinHeader_2.54mm:PinHeader_1x03_P2.54mm_Vertical
- R1: renamed from R?; footprint (none) -> Resistor_THT:R_Axial_DIN0411_L9.9mm_D3.6mm_P15.24mm_Horizontal
- U1, U2, U3, U4: renamed from U?; footprint (none) -> Package_DIP:DIP-14_W7.62mm_LongPads
Connections:
- net p1_chan1: now also U2.3
- net p1_chan2: now also U2.6
- net p1_chan3: now also U2.8
- net p1_chan4: now also U2.11
- net p1_chan5: now also U3.3
- net p1_chan6: now also U3.6
- net p2_chan1: now also U3.8
- net p2_chan2: now also U3.11
- net p2_chan3: now also U4.3
- net p2_chan4: now also U4.6
- net p2_chan5: now also U4.8
- net p2_chan6: now also U4.11
- net at U3.1: now also J3.1; no longer J2.1
- net at U3.4: now also J3.2; no longer J2.2
- net at U2.1: now also J2.1; no longer J3.1
- net at U2.4: now also J2.2; no longer J3.2
- net at U4.1: now also J5.1; no longer J6.1
- net at U4.4: now also J5.2; no longer J6.2
- net at U3.9: now also J6.1; no longer J5.1
- net at U3.12: now also J6.2; no longer J5.2
- net blanking renamed synch
Other:
- moved on the sheet: J1, J2, J3, J4, J5, J6, J7, JP1, R1, U1A, U1G, U2A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
