File: hardware/blanking_board/blanking_board.kicad_sch (KiCad schematic)
At the start: 23 parts

Commit message: update board details
Parts:
- H1, H2, H3, H4: value (none) -> MountingHole; footprint (none) -> MountingHole:MountingHole_3.2mm_M3_ISO7380
- J1, J2, J3, J5, J6, J7, J8: value (none) -> B4B-XH-A_LF__SN_; footprint (none) -> Connector_JST:JST_XH_B4B-XH-A_1x04_P2.50mm_Vertical
- J10, J9: value (none) -> Conn_01x02_Female; footprint (none) -> Connector_JST:JST_XH_B2B-XH-A_1x02_P2.50mm_Vertical
- J11, J12: value (none) -> DB25_Female_MountingHoles; footprint (none) -> Connector_PinHeader_2.54mm:PinHeader_2x13_P2.54mm_Vertical
- J4: value (none) -> B2B-XH-A_LF__SN_; footprint (none) -> Connector_JST:JST_XH_B2B-XH-A_1x02_P2.50mm_Vertical
- JP1: value (none) -> Jumper_NC_Dual; footprint (none) -> Connector_PinHeader_2.54mm:PinHeader_1x03_P2.54mm_Vertical
- R1: value (none) -> 1k; footprint (none) -> Resistor_THT:R_Axial_DIN0411_L9.9mm_D3.6mm_P15.24mm_Horizontal
- U1: value (none) -> 74HC14; footprint (none) -> Package_DIP:DIP-14_W7.62mm_LongPads
- U2, U3, U4: value (none) -> 74LS08; footprint (none) -> Package_DIP:DIP-14_W7.62mm_LongPads
Connections:
- no-connect marks 12 -> 13
